Commit message: Added bot to gazebo simulation.

File: description/lidar.xacro (robot description, xacro)
@@ -4,5 +4,5 @@
         <parent link="chassis" />
         <child link="lidar_frame" />
-        <origin xyz="0.1 0 0.06" rpy="0 0 0" />
+        <origin xyz="0.1 0 0.11" rpy="0 0 0" />
     </joint>
     <link name="lidar_frame">
@@ -11,5 +11,5 @@
                 <cylinder radius="0.057" length="0.07" />
             </geometry>
-            <material name="red" />
+            <material name="magenta" />
         </visual>
         <collision>
@@ -22,3 +22,6 @@
         </xacro:inertial_cylinder>
     </link>
+    <gazebo reference="lidar_frame">
+        <material>Gazebo/Purple</material>
+    </gazebo>
 </robot>

File: description/robot.urdf.xacro (robot description, xacro)
@@ -3,3 +3,4 @@
     <xacro:include filename="robot_core.xacro"/>
     <xacro:include filename="lidar.xacro" />
+    <xacro:include filename="gazebo_control.xacro" />
 </robot>

File: description/robot_core.xacro (robot description, xacro)
@@ -20,4 +20,7 @@
         <color rgba="1 1 0 1"/>
     </material>
+    <material name="magenta">
+        <color rgba="1 0 1 1" />
+    </material>
     <link name="base_link">
     </link>
@@ -30,15 +33,15 @@
     <link name="chassis">
         <visual>
+            <origin xyz="0 0 0.05" />
+            <geometry>
+                <box size="0.266 0.229 0.064" />
+            </geometry>
+            <material name="white" />
+        </visual>
+        <collision>
             <origin xyz="0 0 0" />
             <geometry>
                 <box size="0.266 0.229 0.064" />
             </geometry>
-            <material name="yellow" />
-        </visual>
-        <collision>
-            <origin xyz="0 0 0" />
-            <geometry>
-                <box size="0.266 0.229 0.064" />
-            </geometry>
         </collision>
         <xacro:inertial_box mass="2.0" x="0.266" y="0.229" z="0.064">
@@ -46,9 +49,12 @@
         </xacro:inertial_box>
     </link>
+    <gazebo reference="chassis">
+        <material>Gazebo/White</material>
+    </gazebo>
     <!-- FRONT LEFT WHEEL -->
     <joint name="front_left_wheel_joint" type="continuous">
         <parent link="base_link" />
         <child link="front_left_wheel" />
-        <origin xyz="0.115 0.135 0.07" rpy="-${pi/2} 0 0" />
+        <origin xyz="0.115 0.135 0.12" rpy="-${pi/2} 0 0" />
         <axis xyz="0 0 1" />
     </joint>
@@ -69,9 +75,12 @@
         </xacro:inertial_cylinder>
     </link>
+    <gazebo reference="front_left_wheel">
+        <material>Gazebo/Blue</material>
+    </gazebo>
     <!-- FRONT RIGHT WHEEL -->
     <joint name="front_right_wheel_joint" type="continuous">
         <parent link="base_link" />
         <child link="front_right_wheel" />
-        <origin xyz="0.115 -0.135 0.07" rpy="${pi/2} 0 0" />
+        <origin xyz="0.115 -0.135 0.12" rpy="${pi/2} 0 0" />
         <axis xyz="0 0 -1" />
     </joint>
@@ -92,9 +101,12 @@
         </xacro:inertial_cylinder>
     </link>
+    <gazebo reference="front_right_wheel">
+        <material>Gazebo/Blue</material>
+    </gazebo>
     <!-- BACK LEFT WHEEL -->
     <joint name="back_left_wheel_joint" type="continuous">
         <parent link="base_link" />
         <child link="back_left_wheel" />
-        <origin xyz="-0.115 0.145 0.07" rpy="-${pi/2} 0 0" />
+        <origin xyz="-0.115 0.145 0.12" rpy="-${pi/2} 0 0" />
         <axis xyz="0 0 1" />
     </joint>
@@ -102,22 +114,25 @@
         <visual>
             <geometry>
-                <cylinder radius="0.07" length="0.06" />
-            </geometry>
-            <material name="blue" />
-        </visual>
-        <collision>
-            <geometry>
-                <cylinder radius="0.07" length="0.06" />
-            </geometry>
-        </collision>
-        <xacro:inertial_cylinder mass="0.15" length="0.06" radius="0.07">
-            <origin xyz="0 0 0" rpy="0 0 0" />
-        </xacro:inertial_cylinder>
-    </link>
+                <cylinder radius="0.057" length="0.06" />
+            </geometry>
+            <material name="blue" />
+        </visual>
+        <collision>
+            <geometry>
+                <cylinder radius="0.057" length="0.06" />
+            </geometry>
+        </collision>
+        <xacro:inertial_cylinder mass="0.15" length="0.06" radius="0.057">
+            <origin xyz="0 0 0" rpy="0 0 0" />
+        </xacro:inertial_cylinder>
+    </link>
+    <gazebo reference="back_left_wheel">
+        <material>Gazebo/Blue</material>
+    </gazebo>
     <!-- BACK RIGHT WHEEL -->
     <joint name="back_right_wheel_joint" type="continuous">
         <parent link="base_link" />
         <child link="back_right_wheel" />
-        <origin xyz="-0.115 -0.145 0.07" rpy="${pi/2} 0 0" />
+        <origin xyz="-0.115 -0.145 0.12" rpy="${pi/2} 0 0" />
         <axis xyz="0 0 -1" />
     </joint>
@@ -125,16 +140,68 @@
         <visual>
             <geometry>
-                <cylinder radius="0.07" length="0.06" />
-            </geometry>
-            <material name="blue" />
-        </visual>
-        <collision>
-            <geometry>
-                <cylinder radius="0.07" length="0.06" />
-            </geometry>
-        </collision>
-        <xacro:inertial_cylinder mass="0.15" length="0.06" radius="0.07">
-            <origin xyz="0 0 0" rpy="0 0 0" />
-        </xacro:inertial_cylinder>
-    </link>
+                <cylinder radius="0.057" length="0.06" />
+            </geometry>
+            <material name="blue" />
+        </visual>
+        <collision>
+            <geometry>
+                <cylinder radius="0.057" length="0.06" />
+            </geometry>
+        </collision>
+        <xacro:inertial_cylinder mass="0.15" length="0.06" radius="0.057">
+            <origin xyz="0 0 0" rpy="0 0 0" />
+        </xacro:inertial_cylinder>
+    </link>
+    <gazebo reference="back_right_wheel">
+        <material>Gazebo/Blue</material>
+    </gazebo>
+    <!-- WiFi Antennas-->
+    <joint name="antenna_1_joint" type="fixed">
+        <parent link="base_link" />
+        <child link="antenna_1" />
+        <origin xyz="0.06 0.09 0.18" />
+    </joint>
+    <link name="antenna_1">
+        <visual>
+            <geometry>
+                <cylinder radius="0.007" length="0.18" />
+            </geometry>
+            <material name="white" />
+        </visual>
+        <collision>
+            <geometry>
+                <cylinder radius="0.007" length="0.18" />
+            </geometry>
+        </collision>
+        <xacro:inertial_cylinder mass="0.01" length="0.18" radius="0.007">
+            <origin xyz="0 0 0" rpy="0 0 0" />
+        </xacro:inertial_cylinder>
+    </link>
+    <gazebo reference="antenna_1">
+        <material>Gazebo/White</material>
+    </gazebo>
+    <joint name="antenna_2_joint" type="fixed">
+        <parent link="base_link" />
+        <child link="antenna_2" />
+        <origin xyz="0.03 0.09 0.18" />
+    </joint>
+    <link name="antenna_2">
+        <visual>
+            <geometry>
+                <cylinder radius="0.007" length="0.18" />
+            </geometry>
+            <material name="white" />
+        </visual>
+        <collision>
+            <geometry>
+                <cylinder radius="0.007" length="0.18" />
+            </geometry>
+        </collision>
+        <xacro:inertial_cylinder mass="0.01" length="0.18" radius="0.007">
+            <origin xyz="0 0 0" rpy="0 0 0" />
+        </xacro:inertial_cylinder>
+    </link>
+    <gazebo reference="antenna_2">
+        <material>Gazebo/White</material>
+    </gazebo>
 </robot>
