Commit message: Finished robot body description, simulation working now.

File: description/gazebo_control.xacro (robot description, xacro)
@@ -2,19 +2,29 @@
 <robot xmlns:xacro="http://www.ros.org/wiki/xacro">
    <gazebo>
-        <plugin name="skid_steer_drive_controller" filename="libgazebo_ros_skid_steer_drive.so">
-            <updateRate>100.0</updateRate>
-            <robotNamespace>/</robotNamespace>
-            <leftFrontJoint>front_left_wheel_joint</leftFrontJoint>
-            <rightFrontJoint>front_right_wheel_joint</rightFrontJoint>
-            <leftRearJoint>back_left_wheel_joint</leftRearJoint>
-            <rightRearJoint>back_right_wheel_joint</rightRearJoint>
-            <wheelSeparation>0.23</wheelSeparation>
-            <wheelDiameter>0.13</wheelDiameter>
-            <robotBaseFrame>base_link</robotBaseFrame>
-            <torque>200</torque>
-            <topicName>cmd_vel</topicName>
-            <broadcastTF>true</broadcastTF>
-            <odometryTopic>odom</odometryTopic>
-            <odemetryFrame>odom</odemetryFrame>
+        <plugin name="wheel_drive_controller" filename="libgazebo_ros_diff_drive.so">
+            <!-- wheels -->
+            <num_wheel_pairs>2</num_wheel_pairs>
+            <left_joint>front_left_wheel_joint</left_joint>
+            <left_joint>back_left_wheel_joint</left_joint>
+            <right_joint>front_right_wheel_joint</right_joint>
+            <right_joint>back_right_wheel_joint</right_joint>
+            <!-- kinematics -->
+            <wheel_separation>0.4</wheel_separation>
+            <wheel_diameter>0.1</wheel_diameter>
+            <max_wheel_torque>20.0</max_wheel_torque>
+            <max_wheel_acceleration>10.0</max_wheel_acceleration>
+            <!-- odometry  -->
+            <odometry_source>world</odometry_source>
+            <odometry_frame>odom</odometry_frame>
+            <robot_base_frame>base_link</robot_base_frame>
+            <!-- topic & re remappings -->
+            <ros>
+                <namespace>/</namespace>
+                <argument>/cmd_vel:=cmd_vel</argument>
+                <argument>/odom:=odom</argument>
+            </ros>
+            <publish_odom>true</publish_odom>
+            <publish_odom_tf>true</publish_odom_tf>
+            <update_rate>100.0</update_rate>
         </plugin>
    </gazebo>

File: description/lidar.xacro (robot description, xacro)
@@ -4,5 +4,5 @@
         <parent link="chassis" />
         <child link="lidar_frame" />
-        <origin xyz="0.1 0 0.11" rpy="0 0 0" />
+        <origin xyz="0.1 0 0.08" rpy="0 0 0" />
     </joint>
     <link name="lidar_frame">

File: description/robot_core.xacro (robot description, xacro)
@@ -23,4 +23,11 @@
         <color rgba="1 0 1 1" />
     </material>
+    <link name="world_link">
+    </link>
+    <joint name="world_to_base_joint" type="fixed">
+        <parent link="world_link" />
+        <child link="base_link" />
+        <origin xyz="0 0 0.02" />
+    </joint>
     <link name="base_link">
     </link>
@@ -29,9 +36,9 @@
         <parent link="base_link" />
         <child link="chassis" />
-        <origin xyz="0 0 0.07" />
+        <origin xyz="0 0 0.05" />
     </joint>
     <link name="chassis">
         <visual>
-            <origin xyz="0 0 0.05" />
+            <origin xyz="0 0 0.02" />
             <geometry>
                 <box size="0.266 0.229 0.064" />
@@ -56,5 +63,5 @@
         <parent link="base_link" />
         <child link="front_left_wheel" />
-        <origin xyz="0.115 0.135 0.12" rpy="-${pi/2} 0 0" />
+        <origin xyz="0.115 0.135 0.07" rpy="-${pi/2} 0 0" />
         <axis xyz="0 0 1" />
     </joint>
@@ -82,5 +89,5 @@
         <parent link="base_link" />
         <child link="front_right_wheel" />
-        <origin xyz="0.115 -0.135 0.12" rpy="${pi/2} 0 0" />
+        <origin xyz="0.115 -0.135 0.07" rpy="${pi/2} 0 0" />
         <axis xyz="0 0 -1" />
     </joint>
@@ -108,5 +115,5 @@
         <parent link="base_link" />
         <child link="back_left_wheel" />
-        <origin xyz="-0.115 0.145 0.12" rpy="-${pi/2} 0 0" />
+        <origin xyz="-0.115 0.145 0.07" rpy="-${pi/2} 0 0" />
         <axis xyz="0 0 1" />
     </joint>
@@ -134,5 +141,5 @@
         <parent link="base_link" />
         <child link="back_right_wheel" />
-        <origin xyz="-0.115 -0.145 0.12" rpy="${pi/2} 0 0" />
+        <origin xyz="-0.115 -0.145 0.07" rpy="${pi/2} 0 0" />
         <axis xyz="0 0 -1" />
     </joint>
@@ -160,5 +167,5 @@
         <parent link="base_link" />
         <child link="antenna_1" />
-        <origin xyz="0.06 0.09 0.18" />
+        <origin xyz="0.06 0.09 0.13" />
     </joint>
     <link name="antenna_1">
@@ -184,5 +191,5 @@
         <parent link="base_link" />
         <child link="antenna_2" />
-        <origin xyz="0.03 0.09 0.18" />
+        <origin xyz="0.03 0.09 0.13" />
     </joint>
     <link name="antenna_2">

Commit message: Remodeled minibot description for two-wheel diff drive.

File: description/gazebo_control.xacro (robot description, xacro)
@@ -2,15 +2,12 @@
 <robot xmlns:xacro="http://www.ros.org/wiki/xacro">
    <gazebo>
-        <plugin name="wheel_drive_controller" filename="libgazebo_ros_diff_drive.so">
+        <plugin name="differential_drive_controller" filename="libgazebo_ros_diff_drive.so">
             <!-- wheels -->
-            <num_wheel_pairs>2</num_wheel_pairs>
-            <left_joint>front_left_wheel_joint</left_joint>
-            <left_joint>back_left_wheel_joint</left_joint>
-            <right_joint>front_right_wheel_joint</right_joint>
-            <right_joint>back_right_wheel_joint</right_joint>
+            <left_joint>left_wheel_joint</left_joint>
+            <right_joint>right_wheel_joint</right_joint>
             <!-- kinematics -->
-            <wheel_separation>0.4</wheel_separation>
-            <wheel_diameter>0.1</wheel_diameter>
-            <max_wheel_torque>20.0</max_wheel_torque>
+            <wheel_separation>0.266</wheel_separation>
+            <wheel_diameter>0.16</wheel_diameter>
+            <max_wheel_torque>200.0</max_wheel_torque>
             <max_wheel_acceleration>10.0</max_wheel_acceleration>
             <!-- odometry  -->

File: description/lidar.xacro (robot description, xacro)
@@ -4,20 +4,22 @@
         <parent link="chassis" />
         <child link="lidar_frame" />
-        <origin xyz="0.1 0 0.08" rpy="0 0 0" />
+        <origin xyz="0.225 0 0.2" rpy="0 0 0" />
     </joint>
     <link name="lidar_frame">
         <visual>
+            <origin xyz="0 0 -0.05" />
             <geometry>
-                <cylinder radius="0.057" length="0.07" />
+                <cylinder radius="0.057" length="0.1"/>
             </geometry>
             <material name="magenta" />
         </visual>
         <collision>
+            <origin xyz="0 0 -0.05" />
             <geometry>
-                <cylinder radius="0.057" length="0.04" />
+                <cylinder radius="0.057" length="0.1" />
             </geometry>
         </collision>
-        <xacro:inertial_cylinder mass="0.1" length="0.04" radius="0.057">
-            <origin xyz="0 0 0" rpy="0 0 0" />
+        <xacro:inertial_cylinder mass="0.1" length="0.1" radius="0.057">
+            <origin xyz="0 0 -0.05" rpy="0 0 0" />
         </xacro:inertial_cylinder>
     </link>
@@ -36,5 +38,5 @@
                 </scan>
                 <range>
-                    <min>0.4 </min>
+                    <min>0.2 </min>
                     <max> 12 </max>
                 </range>

File: description/robot_core.xacro (robot description, xacro)
@@ -1,4 +1,10 @@
 <?xml version="1.0"?>
 <robot xmlns:xacro="http://www.ros.org/wiki/xacro">
+    <!-- EDIT ROBOT DESCRIPTION HERE -->
+    <xacro:property name="chassis_width" value="0.05" />
+    <xacro:property name="chassis_length" value="0.266" />
+    <xacro:property name="chassis_height" value="0.05" />
+    <xacro:property name="wheel_radius" value="0.08" />
+    <xacro:property name="wheel_thickness" value="0.04" />
     <xacro:include filename="inertial_macros.xacro" />
     <material name="white">
@@ -45,22 +51,22 @@
         <parent link="base_link" />
         <child link="chassis" />
-        <origin xyz="0 0 0.05" />
+        <origin xyz="0 0 0" />
     </joint>
     <link name="chassis">
         <visual>
-            <origin xyz="0 0 0.02" />
+            <origin xyz="0 0 ${wheel_radius}" />
             <geometry>
-                <box size="0.266 0.229 0.064" />
+                <box size="${chassis_width} ${chassis_length} ${chassis_height}" />
             </geometry>
             <material name="white" />
         </visual>
         <collision>
-            <origin xyz="0 0 0" />
+            <origin xyz="0 0 ${wheel_radius/2}" />
             <geometry>
-                <box size="0.266 0.229 0.064" />
+                <box size="${chassis_width} ${chassis_length} ${chassis_height}" />
             </geometry>
         </collision>
-        <xacro:inertial_box mass="2.0" x="0.266" y="0.229" z="0.064">
-            <origin xyz="0 0 0" rpy="0 0 0" />
+        <xacro:inertial_box mass="2.0" x="${chassis_width}" y="${chassis_length}" z="${chassis_height}">
+            <origin xyz="0 0 ${wheel_radius}" rpy="0 0 0" />
         </xacro:inertial_box>
     </link>
@@ -68,15 +74,41 @@
         <material>Gazebo/White</material>
     </gazebo>
-    <!-- FRONT LEFT WHEEL -->
-    <joint name="front_left_wheel_joint" type="continuous">
+    <joint name="chassis2_joint" type="fixed">
+        <parent link="chassis" />
+        <child link="chassis2" />
+        <origin xyz="0 0 0" />
+    </joint>
+    <link name="chassis2">
+        <visual>
+            <origin xyz="0.133 0 ${wheel_radius}" />
+            <geometry>
+                <box size="${chassis_length} ${chassis_width} ${chassis_height}" />
+            </geometry>
+            <material name="white" />
+        </visual>
+        <collision>
+            <origin xyz="0 0 ${wheel_radius/2}" />
+            <geometry>
+                <box size="${chassis_length} ${chassis_width} ${chassis_height}" />
+            </geometry>
+        </collision>
+        <xacro:inertial_box mass="2.0" x="${chassis_length}" y="${chassis_width}" z="${chassis_height}">
+            <origin xyz="0.133 0 ${wheel_radius}" rpy="0 0 0" />
+        </xacro:inertial_box>
+    </link>
+    <gazebo reference="chassis2">
+        <material>Gazebo/White</material>
+    </gazebo>
+    <!-- RIGHT WHEEL LINK -->
+    <joint name="right_wheel_joint" type="continuous">
         <parent link="base_link" />
-        <child link="front_left_wheel" />
-        <origin xyz="0.115 0.135 0.07" rpy="-${pi/2} 0 0" />
-        <axis xyz="0 0 1" />
+        <child link="right_wheel" />
+        <origin xyz="0 ${chassis_length/2} ${wheel_radius}" rpy="${pi/2} 0 0" />
+        <axis xyz="0 0 1"/>
     </joint>
-    <link name="front_left_wheel">
+    <link name="right_wheel">
         <visual>
             <geometry>
-                <cylinder radius="0.057" length="0.04" />
+                <cylinder radius="${wheel_radius}" length="${wheel_thickness}" />
             </geometry>
             <material name="blue" />
@@ -84,25 +116,27 @@
         <collision>
             <geometry>
-                <cylinder radius="0.057" length="0.04" />
+                <cylinder radius="${wheel_radius}" length="${wheel_thickness}" />
             </geometry>
         </collision>
-        <xacro:inertial_cylinder mass="0.1" length="0.04" radius="0.057">
+        <xacro:inertial_cylinder mass="0.5" length="${wheel_thickness}" radius="${wheel_radius}">
             <origin xyz="0 0 0" rpy="0 0 0" />
         </xacro:inertial_cylinder>
     </link>
-    <gazebo reference="front_left_wheel">
+    <gazebo reference="right_wheel">
         <material>Gazebo/Blue</material>
+        <mu1 value="3" />
+        <mu2 value="3" />
     </gazebo>
-    <!-- FRONT RIGHT WHEEL -->
-    <joint name="front_right_wheel_joint" type="continuous">
+    <!-- LEFT WHEEL LINK -->
+    <joint name="left_wheel_joint" type="continuous">
         <parent link="base_link" />
-        <child link="front_right_wheel" />
-        <origin xyz="0.115 -0.135 0.07" rpy="${pi/2} 0 0" />
-        <axis xyz="0 0 -1" />
+        <child link="left_wheel" />
+        <origin xyz="0 ${-chassis_length/2} ${wheel_radius}" rpy="-${pi/2} 0 0" />
+        <axis xyz="0 0 -1"/>
     </joint>
-    <link name="front_right_wheel">
+    <link name="left_wheel">
         <visual>
             <geometry>
-                <cylinder radius="0.057" length="0.04" />
+                <cylinder radius="${wheel_radius}" length="${wheel_thickness}" />
             </geometry>
             <material name="blue" />
@@ -110,114 +144,39 @@
         <collision>
             <geometry>
-                <cylinder radius="0.057" length="0.04" />
+                <cylinder radius="${wheel_radius}" length="${wheel_thickness}" />
             </geometry>
         </collision>
-        <xacro:inertial_cylinder mass="0.1" length="0.04" radius="0.057">
+        <xacro:inertial_cylinder mass="0.5" length="${wheel_thickness}" radius="${wheel_radius}">
             <origin xyz="0 0 0" rpy="0 0 0" />
         </xacro:inertial_cylinder>
     </link>
-    <gazebo reference="front_right_wheel">
+    <gazebo reference="left_wheel">
         <material>Gazebo/Blue</material>
+        <mu1 value="3" />
+        <mu2 value="3" />
     </gazebo>
-    <!-- BACK LEFT WHEEL -->
-    <joint name="back_left_wheel_joint" type="continuous">
-        <parent link="base_link" />
-        <child link="back_left_wheel" />
-        <origin xyz="-0.115 0.145 0.07" rpy="-${pi/2} 0 0" />
-        <axis xyz="0 0 1" />
+    <!-- CASTER WHEEL LINK -->
+    <joint name="caster_wheel_joint" type="fixed">
+        <parent link="chassis" />
+        <child link="caster_wheel" />
+        <origin xyz="0.225 0 0.05" />
     </joint>
-    <link name="back_left_wheel">
+    <link name="caster_wheel" >
         <visual>
             <geometry>
-                <cylinder radius="0.057" length="0.06" />
+                <sphere radius="0.05"/>
             </geometry>
-            <material name="blue" />
+            <material name="black" />
         </visual>
         <collision>
             <geometry>
-                <cylinder radius="0.057" length="0.06" />
+                <sphere radius="0.05"/>
             </geometry>
         </collision>
-        <xacro:inertial_cylinder mass="0.15" length="0.06" radius="0.057">
-            <origin xyz="0 0 0" rpy="0 0 0" />
-        </xacro:inertial_cylinder>
     </link>
-    <gazebo reference="back_left_wheel">
-        <material>Gazebo/Blue</material>
-    </gazebo>
-    <!-- BACK RIGHT WHEEL -->
-    <joint name="back_right_wheel_joint" type="continuous">
-        <parent link="base_link" />
-        <child link="back_right_wheel" />
-        <origin xyz="-0.115 -0.145 0.07" rpy="${pi/2} 0 0" />
-        <axis xyz="0 0 -1" />
-    </joint>
-    <link name="back_right_wheel">
-        <visual>
-            <geometry>
-                <cylinder radius="0.057" length="0.06" />
-            </geometry>
-            <material name="blue" />
-        </visual>
-        <collision>
-            <geometry>
-                <cylinder radius="0.057" length="0.06" />
-            </geometry>
-        </collision>
-        <xacro:inertial_cylinder mass="0.15" length="0.06" radius="0.057">
-            <origin xyz="0 0 0" rpy="0 0 0" />
-        </xacro:inertial_cylinder>
-    </link>
-    <gazebo reference="back_right_wheel">
-        <material>Gazebo/Blue</material>
-    </gazebo>
-    <!-- WiFi Antennas-->
-    <joint name="antenna_1_joint" type="fixed">
-        <parent link="base_link" />
-        <child link="antenna_1" />
-        <origin xyz="0.06 0.09 0.13" />
-    </joint>
-    <link name="antenna_1">
-        <visual>
-            <geometry>
-                <cylinder radius="0.007" length="0.18" />
-            </geometry>
-            <material name="white" />
-        </visual>
-        <collision>
-            <geometry>
-                <cylinder radius="0.007" length="0.18" />
-            </geometry>
-        </collision>
-        <xacro:inertial_cylinder mass="0.01" length="0.18" radius="0.007">
-            <origin xyz="0 0 0" rpy="0 0 0" />
-        </xacro:inertial_cylinder>
-    </link>
-    <gazebo reference="antenna_1">
-        <material>Gazebo/White</material>
-    </gazebo>
-    <joint name="antenna_2_joint" type="fixed">
-        <parent link="base_link" />
-        <child link="antenna_2" />
-        <origin xyz="0.03 0.09 0.13" />
-    </joint>
-    <link name="antenna_2">
-        <visual>
-            <geometry>
-                <cylinder radius="0.007" length="0.18" />
-            </geometry>
-            <material name="white" />
-        </visual>
-        <collision>
-            <geometry>
-                <cylinder radius="0.007" length="0.18" />
-            </geometry>
-        </collision>
-        <xacro:inertial_cylinder mass="0.01" length="0.18" radius="0.007">
-            <origin xyz="0 0 0" rpy="0 0 0" />
-        </xacro:inertial_cylinder>
-    </link>
-    <gazebo reference="antenna_2">
-        <material>Gazebo/White</material>
+    <gazebo reference="caster_wheel">
+        <material>Gazebo/Black</material>
+        <mu1 value="0.001" />
+        <mu2 value="0.001" />
     </gazebo>
 </robot>

File: description/ros2_control.xacro (robot description, xacro)
@@ -5,32 +5,16 @@
             <plugin>gazebo_ros2_control/GazeboSystem</plugin>
         </hardware>
-        <joint name="front_left_wheel_joint">
+        <joint name="left_wheel_joint">
             <command_interface name="velocity">
-                <param name="min">-10</param>
-                <param name="max">10</param>
+                <param name="min">-100</param>
+                <param name="max">100</param>
             </command_interface>
             <state_interface name="velocity" />
             <state_interface name="position" />
         </joint>
-        <joint name="front_right_wheel_joint">
+        <joint name="right_wheel_joint">
             <command_interface name="velocity">
-                <param name="min">-10</param>
-                <param name="max">10</param>
-            </command_interface>
-            <state_interface name="velocity" />
-            <state_interface name="position" />
-        </joint>
-        <joint name="back_left_wheel_joint">
-            <command_interface name="velocity">
-                <param name="min">-10</param>
-                <param name="max">10</param>
-            </command_interface>
-            <state_interface name="velocity" />
-            <state_interface name="position" />
-        </joint>
-        <joint name="back_right_wheel_joint">
-            <command_interface name="velocity">
-                <param name="min">-10</param>
-                <param name="max">10</param>
+                <param name="min">-100</param>
+                <param name="max">100</param>
             </command_interface>
             <state_interface name="velocity" />
